File: Hardware/Hardware.kicad_pcb (KiCad board)
At the start: 2 copper layers, 7 parts, among them J1 Conn_01x11_Pin, SW1 SW_Push, SW2 SW_Push, SW3 SW_Push, SW4 SW_Push, U1 ESP32-C3_SUPERMINI_TH, U2 DM-OLED096-636

Commit message: feat: add routes
Parts:
- removed SW1, SW2, SW3, SW4: SW_Push, Button_Switch_THT:SW_PUSH_6mm
- added C1: 100nF, Capacitor_SMD:C_0603_1608Metric_Pad1.08x0.95mm_HandSolder, F.Cu at (73.8, 54.4)
- added C2: 100nF, Capacitor_SMD:C_0603_1608Metric_Pad1.08x0.95mm_HandSolder, F.Cu at (73.8, 57.6)
- added C3: 100nF, Capacitor_SMD:C_0603_1608Metric_Pad1.08x0.95mm_HandSolder, F.Cu at (91.8, 55.2)
- added C4: 100nF, Capacitor_SMD:C_0603_1608Metric_Pad1.08x0.95mm_HandSolder, F.Cu at (91.8, 56.9)
- added C5: 100nF, Capacitor_SMD:C_0603_1608Metric_Pad1.08x0.95mm_HandSolder, F.Cu at (73.8, 56.0)
- added S1: JS1400AFQ, footprints:SW_JS1400AFQ, F.Cu at (82.8, 56.0)
- added kibuzzard-6891AAE2: G***, kibuzzard-6891AAE2, B.Cu at (71.0, 27.5)
- added kibuzzard-6891AB0F: G***, kibuzzard-6891AB0F, B.Cu at (71.0, 30.1)
- added kibuzzard-6891AB20: G***, kibuzzard-6891AB20, B.Cu at (71.0, 35.3)
- added kibuzzard-6891AB27: G***, kibuzzard-6891AB27, B.Cu at (70.9, 32.5)
- added kibuzzard-6891AB30: G***, kibuzzard-6891AB30, B.Cu at (71.0, 38.0)
- added kibuzzard-6891AB39: G***, kibuzzard-6891AB39, B.Cu at (71.0, 40.4)
- added kibuzzard-6891AB3F: G***, kibuzzard-6891AB3F, B.Cu at (71.0, 42.8)
- added kibuzzard-6891AB44: G***, kibuzzard-6891AB44, B.Cu at (71.0, 45.8)
- added kibuzzard-6891AB4C: G***, kibuzzard-6891AB4C, B.Cu at (71.0, 48.1)
- added kibuzzard-6891AB56: G***, kibuzzard-6891AB56, B.Cu at (71.0, 50.6)
- J1: value Conn_01x11_Pin -> Conn_01x10_Socket; footprint Connector_PinHeader_2.54mm:PinHeader_1x11_P2.54mm_Vertical -> Connector_PinHeader_2.54mm:PinHeader_1x10_P2.54mm_Vertical
- moved U1 57.2 mm to (87.3, 37.5), turned to 90 degrees
- moved J1 29.3 mm to (67.3, 50.4)
- moved U2 2.31 mm to (82.6, 36.4)
Connections:
- net /GPIO20 renamed /RX
- net /GPIO5 renamed /MISO
- net /GPIO6 renamed /MOSI
- net /GPIO7 renamed /SS
- net /GPIO8 renamed /SDA
- net /GPIO9 renamed /SCL
- J1 pad 10: +3V3 -> GND
- J1 pad 7: /GPIO10 -> /TX
- J1 pad 9: /GPIO21 -> +3V3
- U1 pad 0: /BTN1 -> /F1
- U1 pad 1: /BTN2 -> /F2
- U1 pad 10: /GPIO10 -> /F5
- U1 pad 2: /BTN3 -> /F4
- U1 pad 21: /GPIO21 -> /TX
- U1 pad 3: /BTN4 -> /F3
Routing:
- net /CLK: track 0.00 -> 77.6 mm
- net /SDA: track 0.00 -> 58.5 mm, vias 0 -> 1
- net /F1: track 0.00 -> 56.8 mm, vias 0 -> 1
- net /SCL: track 0.00 -> 56.7 mm, vias 0 -> 1
- net /MISO: track 0.00 -> 51.2 mm
- net /F3: track 0.00 -> 50.9 mm, vias 0 -> 1
- net /MOSI: track 0.00 -> 40.0 mm
- net /F4: track 0.00 -> 40.0 mm, vias 0 -> 1
- net /SS: track 0.00 -> 38.4 mm
- net /F2: track 0.00 -> 35.5 mm, vias 0 -> 1
- net +3V3: track 0.00 -> 32.9 mm
- net /RX: track 0.00 -> 26.6 mm
- net /TX: track 0.00 -> 26.5 mm
- net /F5: track 0.00 -> 17.1 mm, vias 0 -> 1
- net GND: vias 0 -> 31
- added copper zone on B.Cu, net GND
- added copper zone on F.Cu, net GND
Other:
- board outline added: 35 x 40 mm
