File: Hardware/Hardware.kicad_pcb (KiCad board)
At the start: 2 copper layers, 35 x 40 mm, 19 parts, among them J1 Conn_01x10_Socket, U1 ESP32-C3_SUPERMINI_TH, U2 DM-OLED096-636

Commit message: feat: add open hardware logo & version
Parts:
- added G***: LOGO, footprints:open_hardware, B.Cu at (73.3, 57.0)
- added kibuzzard-689394AC: G***, kibuzzard-689394AC, B.Cu at (92.1, 58.7)
Other:
- board text added: "Design by: Adonai Diaz"
